Commit message: add controller with keyboard + modified graph

File: mybot_gazebo_tutorial/mybot_description/urdf/macros.xacro (robot description, xacro)
@@ -58,5 +58,5 @@
           k_velocity="0" />
         <joint_properties damping="0.5" friction="0.5"/>
-        <limit lower="0.6" upper="0.6" effort="10000.0" velocity="10.0"/>
+        <limit lower="-0.6" upper="0.6" effort="10000.0" velocity="10.0"/>
       </joint>
       <transmission name="${st}_trans">
@@ -73,4 +73,5 @@
         <mu1>0.3</mu1>
         <mu2>0.3</mu2>
+        <self_collide>1</self_collide>
       </gazebo>
     </macro>
@@ -117,5 +118,4 @@
         </collision>
       </link>
-      <!-- ${ch}_joint -->
       <joint
         name="${ch}_joint"
@@ -133,5 +133,5 @@
           k_velocity="0" />
         <joint_properties damping="0.0" friction="0.0"/>
-        <limit lower="0.4" upper="0.4" effort="10000.0" velocity="10.0"/>
+        <limit lower="-0.4" upper="0.4" effort="10000.0" velocity="10.0"/>
       </joint>
       <transmission name="${ch}_trans">
@@ -148,4 +148,5 @@
         <mu1>0.3</mu1>
         <mu2>0.3</mu2>
+        <self_collide>1</self_collide>
       </gazebo>
     </macro>
@@ -208,5 +209,5 @@
           k_velocity="0" />
         <joint_properties damping="0.0" friction="0.0"/>
-        <limit lower="0.4" upper="0.4" effort="10000.0" velocity="10.0"/>
+        <limit lower="-0.4" upper="0.4" effort="10000.0" velocity="10.0"/>
       </joint>
       <!-- transmission -->
@@ -225,4 +226,5 @@
         <mu1>0.3</mu1>
         <mu2>0.3</mu2>
+        <self_collide>1</self_collide>
       </gazebo>
     </macro>
@@ -275,13 +277,9 @@
           xyz="${xyz_ori_joint}"
           rpy="${rpy_ori_joint}" />
-        <parent
-          link="${pr}_Link" />
-        <child
-          link="${ch}_Link" />
-        <axis
-          xyz="0 0 1" />
+        <parent link="${pr}_Link" />
+        <child link="${ch}_Link" />
+        <axis xyz="0 0 1" />
         <limit effort="10000.0" velocity="100.0"/>
-        <safety_controller
-          k_velocity="0" />
+        <safety_controller k_velocity="0" />
         <joint_properties damping="0.0" friction="0.0"/>
       </joint>
@@ -300,7 +298,10 @@
         <mu2 value="1.0"/>
         <kp  value="10000000.0" />
-        <kd  value="1.0" />
+        <kd>100.0</kd>
         <fdir1 value="1 0 0"/>
+        <minDepth>0.001</minDepth>
+        <maxVel>1.0</maxVel>
         <material>Gazebo/Black</material>
+        <self_collide>1</self_collide>
       </gazebo>
     </macro>

File: mybot_gazebo_tutorial/mybot_description/urdf/mybot.xacro (robot description, xacro)
@@ -29,5 +29,5 @@
         rpy="0 0 0" />
       <mass
-        value="10.9977" />
+        value="1.9977" />
       <inertia
         ixx="0.41015032534565"
@@ -99,5 +99,5 @@
   </link>
   <joint name="Pivot_mid_joint"
-    type="fixed">
+    type="revolute">
     <origin
       xyz="-0.0147751266463989 0 0.117"
@@ -111,5 +111,10 @@
     <safety_controller
       k_velocity="0" />
-  </joint>
+    <joint_properties damping="0.0" friction="0.0"/>
+    <limit lower="-0.4" upper="0.4" effort="10000.0" velocity="10.0"/>
+  </joint>
+  <gazebo reference="Pivot_mid_Link">
+    <self_collide>1</self_collide>
+  </gazebo>
   <!-- camera front -->
   <joint name="camera_joint_front" type="fixed">
